File: LED_Heart.sch (EAGLE design)
At the start: 30 parts, among them J1 AVR_SPI_PRG_6PTH, U1 ATmega328P-AU

Commit message: Cleanup of schematic
Parts:
- C1: value (none) -> 0.1uf
- C2: value (none) -> 470pf
- R1, R10, R11, R2, R3, R4, R5, R6, R7, R8, R9: value (none) -> 220
- R12, R17: value (none) -> 10k
- XTAL: value (none) -> CSTCE16M0V53-R0 16MHZ
Connections:
- removed net N$37: J1.6, LED0.C, LED1.C, LED10.C, LED2.C, LED3.C, LED4.C, LED5.C, LED6.C, LED7.C, LED8.C, LED9.C
- net GND: now also J1.6, LED0.C, LED1.C, LED10.C, LED2.C, LED3.C, LED4.C, LED5.C, LED6.C, LED7.C, LED8.C, LED9.C
Other:
- moved on the sheet: C1
